File: Hardware/LuminX WLED.kicad_pcb (KiCad board)
At the start: 4 copper layers, 94.6 x 64.6 mm, 97 parts, among them J1 USB_C_Receptacle_USB2.0, J2 5mm Screw Terminal, J3 USB_B_Micro, J4 Conn_01x04_Pin, J5 Barrel_Jack_Switch, J7 5mm Screw Terminal, J8 5mm Screw Terminal, J9 Conn_01x03_Pin, K1 G5LE-1, Q1 BC847, Q2 BC847, Q3 BC847, Q5 IRF5305, SW2 SW_Push, SW3 SW_Push, U1 CH340G, U10 INA180A1, U2 USBLC6-2P6, U3 ESP32-WROOM-32D, U4 TSOP382xx, U6 AP2112K-3.3, U7 DS18B20, U8 74AHCT244, U9 TPS54332, Y1 12MHz

Commit message: v1.0
Parts:
- removed REF**: OSHW-Symbol_6.7x6mm_SilkScreen, Symbol:OSHW-Symbol_6.7x6mm_SilkScreen
