File: Hardware/LuminX WLED.kicad_sch (KiCad schematic)
At the start: 4 parts

Commit message: v1.0
Parts:
- H1, H2, H3, H4: now left out of the parts list
Changed lines of the file:
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@@
   )
   (symbol (lib_id "Mechanical:MountingHole_Pad") (at 273.685 171.45 0) (unit 1)
-    (in_bom yes) (on_board yes) (dnp no) (fields_autoplaced)
+    (in_bom no) (on_board yes) (dnp no) (fields_autoplaced)
     (property "Reference" "H1" (at 276.225 170.6153 0)
       (effects (font (size 1.27 1.27)) (justify left) hide)
@@
   )
   (symbol (lib_id "Mechanical:MountingHole_Pad") (at 268.605 171.45 0) (unit 1)
-    (in_bom yes) (on_board yes) (dnp no) (fields_autoplaced)
+    (in_bom no) (on_board yes) (dnp no) (fields_autoplaced)
     (property "Reference" "H4" (at 271.145 170.6153 0)
       (effects (font (size 1.27 1.27)) (justify left) hide)
@@
   )
   (symbol (lib_id "Mechanical:MountingHole_Pad") (at 278.765 171.45 0) (unit 1)
-    (in_bom yes) (on_board yes) (dnp no) (fields_autoplaced)
+    (in_bom no) (on_board yes) (dnp no) (fields_autoplaced)
     (property "Reference" "H3" (at 281.305 170.6153 0)
       (effects (font (size 1.27 1.27)) (justify left) hide)
@@
   )
   (symbol (lib_id "Mechanical:MountingHole_Pad") (at 263.525 171.45 0) (unit 1)
-    (in_bom yes) (on_board yes) (dnp no) (fields_autoplaced)
+    (in_bom no) (on_board yes) (dnp no) (fields_autoplaced)
     (property "Reference" "H2" (at 266.065 170.6153 0)
       (effects (font (size 1.27 1.27)) (justify left) hide)
