File: Hardware/LuminX Pro.kicad_pcb (KiCad board)
At the start: 4 copper layers, 94.6 x 64.6 mm, 96 parts, among them J1 USB_C_Receptacle_USB2.0, J2 5mm Screw Terminal, J3 USB_B_Micro, J4 Conn_01x04_Pin, J5 Barrel_Jack_Switch, J7 5mm Screw Terminal, J8 5mm Screw Terminal, J9 Conn_01x03_Pin, K1 G5LE-1, Q1 BC847, Q2 BC847, Q3 BC847, Q5 IRF5305, SW2 SW_Push, SW3 SW_Push, U1 CH340G, U10 INA180A1, U2 USBLC6-2P6, U3 ESP32-WROOM-32D, U4 TSOP382xx, U6 AP2112K-3.3, U7 DS18B20, U8 74AHCT244, U9 TPS54332, Y1 12MHz

Commit message: Revise v2 schematic
Parts:
- removed BOOT1, SW2, SW3: SW_Push, Button_Switch_SMD:SW_SPST_PTS645
- removed C22: 10u, Capacitor_SMD:C_1206_3216Metric
- removed C23: 100n, Capacitor_SMD:C_0603_1608Metric
- removed C24, C25: 22u, Capacitor_SMD:C_1206_3216Metric
- removed D10: SS34, Diode_SMD:D_SMA
- removed D11, D13, D14: SD05, Diode_SMD:D_SOD-323
- removed D12: SS54, Diode_SMD:D_SMA
- removed D9: AMBER, LED_SMD:LED_1206_3216Metric_ReverseMount_Hole1.8x2.4mm
- removed J7: 5mm Screw Terminal, TerminalBlock_Phoenix:TerminalBlock_Phoenix_MKDS-1,5-2_1x02_P5.00mm_Horizontal
- removed J8: 5mm Screw Terminal, TerminalBlock_Phoenix:TerminalBlock_Phoenix_MKDS-1,5-4_1x04_P5.00mm_Horizontal
- removed J9: Conn_01x03_Pin, Connector_PinHeader_2.54mm:PinHeader_1x03_P2.54mm_Vertical
- removed L2: 10u/3A, Inductor_SMD:L_Sunlord_SWPA8040S
- removed Q5: IRF5305, Package_TO_SOT_SMD:TO-252-2
- removed R21: 10k, Resistor_SMD:R_0603_1608Metric
- removed R22: 1k2, Resistor_SMD:R_0603_1608Metric
- removed R23: 680, Resistor_SMD:R_0603_1608Metric
- removed U10: INA180A1, Package_TO_SOT_SMD:SOT-23-5
- removed U9: TPS54332, Package_SO:SOIC-8_3.9x4.9mm_P1.27mm
- added C10: 10u, Capacitor_SMD:C_1206_3216Metric, F.Cu at (59.3, 109.9)
- added C11: 10u, Capacitor_SMD:C_1206_3216Metric, F.Cu at (62.2, 107.2)
- added F2: 750mA, Fuse:Fuse_1206_3216Metric, F.Cu at (114.0, 77.5)
- added F3: Fuse, Fuse:Fuseholder_Clip-5x20mm_Littelfuse_521_Lateral_P17.00x5.00mm_D1.30mm_Horizontal, F.Cu at (57.3, 110.6)
- added H5: MountingHole, MountingHole:MountingHole_3.2mm_M3_Pad_Via, F.Cu at (211.0, 74.5)
- added H6: MountingHole, MountingHole:MountingHole_3.2mm_M3_Pad_Via, F.Cu at (211.0, 82.5)
- added H7: MountingHole, MountingHole:MountingHole_3.2mm_M3_Pad_Via, F.Cu at (211.0, 90.5)
- added H8: MountingHole, MountingHole:MountingHole_3.2mm_M3_Pad_Via, F.Cu at (211.0, 98.4)
- added J6: Phoenix MKDS x8 5mm, TerminalBlock_Phoenix:TerminalBlock_Phoenix_MKDS-1,5-8_1x08_P5.00mm_Horizontal, F.Cu at (105.7, 109.8)
- added L1: 10u/2A, Inductor_SMD:L_Sunlord_MWSA0603S, F.Cu at (90.6, 148.8)
- added SW_C1: SW_Push, Button_Switch_SMD:SW_SPST_PTS645, F.Cu at (148.6, 120.0)
- added SW_L1: SW_Push, Button_Switch_SMD:SW_SPST_PTS645, F.Cu at (136.6, 120.0)
- added SW_R1: SW_Push, Button_Switch_SMD:SW_SPST_PTS645, F.Cu at (160.6, 120.0)
- added U5: ESP32-WROOM-32D, RF_Module:ESP32-WROOM-32D, F.Cu at (148.6, 81.6)
- C1: value 100n -> 30p
- C12: value 1u -> 100n
- C13: value 1u -> 10u; footprint Capacitor_SMD:C_0603_1608Metric -> Capacitor_SMD:C_0805_2012Metric
- C14: value 100n -> 47p
- C15, C16: value 100n -> 22u; footprint Capacitor_SMD:C_0603_1608Metric -> Capacitor_SMD:C_1206_3216Metric
- C19: value 10p -> 1u
- C20: value 1n -> 1u
- C21: value 8n2 -> 1000u; footprint Capacitor_SMD:C_0603_1608Metric -> Capacitor_THT:CP_Radial_D12.5mm_P5.00mm
- C3: value 10u -> 30p; footprint Capacitor_SMD:C_0805_2012Metric -> Capacitor_SMD:C_0603_1608Metric
- C4: value 30p -> 100n; moved to B.Cu
- C5: value 30p -> 2u2; footprint Capacitor_SMD:C_0603_1608Metric -> Capacitor_SMD:C_0805_2012Metric
- C7: value 100u/35V -> 10u; footprint Capacitor_THT:CP_Radial_D6.3mm_P2.50mm -> Capacitor_SMD:C_0805_2012Metric
- C8: value 10u -> 10n; footprint Diode_SMD:D_0805_2012Metric -> Capacitor_SMD:C_0603_1608Metric
- C9: value 1000u -> 100n; footprint Capacitor_THT:CP_Radial_D12.5mm_P5.00mm -> Capacitor_SMD:C_0603_1608Metric
- D1: value SS34 -> US1G
- D2: value SD05 -> SS34; footprint Diode_SMD:D_SOD-323 -> Diode_SMD:D_SMA; moved to B.Cu
- D3: value US1G -> GREEN; footprint Diode_SMD:D_SMA -> LED_SMD:LED_0805_2012Metric
- D4: value YELLOW -> AMBER; footprint LED_SMD:LED_1206_3216Metric_ReverseMount_Hole1.8x2.4mm -> LED_SMD:LED_0805_2012Metric
- D5, D6: value GREEN -> SP0502BAHT; footprint LED_SMD:LED_1206_3216Metric_ReverseMount_Hole1.8x2.4mm -> Package_TO_SOT_SMD:SOT-23
- D7: value SD05 -> US1G; footprint Diode_SMD:D_SOD-323 -> Diode_SMD:D_SMA
- F1: value 10A -> 3.5A; footprint Fuse:Fuseholder_Blade_Mini_Keystone_3568 -> Fuse:Fuse_1206_3216Metric
- FB1: value 100R -> 120R
- J1: value USB_C_Receptacle_USB2.0 -> GCT USB4105; footprint Connector_USB:USB_C_Receptacle_HRO_TYPE-C-31-M-12 -> Connector_USB:USB_C_Receptacle_GCT_USB4105-xx-A_16P_TopMnt_Horizontal
- J2: value 5mm Screw Terminal -> JST PH; footprint TerminalBlock_Phoenix:TerminalBlock_Phoenix_MKDS-1,5-2_1x02_P5.00mm_Horizontal -> Connector_JST:JST_PH_B4B-PH-SM4-TB_1x04-1MP_P2.00mm_Vertical
- J3: value USB_B_Micro -> JST PH; footprint Connector_USB:USB_Micro-B_Molex-105017-0001 -> Connector_JST:JST_PH_B4B-PH-SM4-TB_1x04-1MP_P2.00mm_Vertical
- J4: value Conn_01x04_Pin -> GCT DCJ200-10; footprint Connector_JST:JST_SH_BM04B-SRSS-TB_1x04-1MP_P1.00mm_Vertical -> MG_Footprint_Lib:Conn_BarrelJack_GCT_DCJ200-10-A_Horizontal
- J5: value Barrel_Jack_Switch -> 5mm Screw Terminal; footprint Connector_BarrelJack:BarrelJack_Horizontal -> TerminalBlock_Phoenix:TerminalBlock_Phoenix_MKDS-1,5-2_1x02_P5.00mm_Horizontal
- MK1: value INMP441 -> MIC_I2S_INMP441; footprint Package_DIP:DIP-6_W7.62mm_Socket -> MG_Footprint_Lib:MIC_I2S_ICS-43434+INMP441
- R1: value 5k1 -> 0R
- R10: value 470R -> 220R
- R11: value 1k -> 100k
- R12: value 10k -> 13k7
- R13: value 1k -> 4k7
- R14: value 0.1R -> 4k7; footprint Resistor_SMD:R_1206_3216Metric -> Resistor_SMD:R_0603_1608Metric
- R15: value 4k7 -> 10k
- R16: value 1k -> 10k
- R19: value 4k7 -> 470R
- R2: value 5k1 -> 10k
- R20: value 33k -> 1k
- R3, R4: value 470R -> 5k1
- R6, R7: value 10k -> 470R
- U1: value CH340G -> ~; footprint Package_SO:SOIC-16_3.9x9.9mm_P1.27mm -> MG_Footprint_Lib:Vishay_IR_Heimdall
- U2: value USBLC6-2P6 -> DS18B20; footprint Package_TO_SOT_SMD:SOT-666 -> Package_TO_SOT_THT:TO-92_Inline
- U3: value ESP32-WROOM-32D -> CH340G; footprint RF_Module:ESP32-WROOM-32D -> Package_SO:SOIC-16_3.9x9.9mm_P1.27mm
- U4: value TSOP382xx -> USBLC6-2P6; footprint OptoDevice:Vishay_MINICAST-3Pin -> Package_TO_SOT_SMD:SOT-666; moved to F.Cu
- U6: value AP2112K-3.3 -> TPS54302; footprint Package_TO_SOT_SMD:SOT-23-5 -> Package_TO_SOT_SMD:SOT-23-6
- U7: value DS18B20 -> 74AHCT125; footprint Package_TO_SOT_THT:TO-92_Inline -> Package_SO:SO-14_3.9x8.65mm_P1.27mm; moved to F.Cu
- U8: value 74AHCT244 -> AP2112K-3.3; footprint Package_SO:TSSOP-20_4.4x6.5mm_P0.65mm -> Package_TO_SOT_SMD:SOT-23-5
- moved C5 179.5 mm to (290.9, 58.2), turned to 0 degrees
- moved J3 120.9 mm to (209.4, 55.2), turned to 0 degrees
- moved C7 104.6 mm to (221.2, 93.2), turned to 0 degrees
- moved U6 104.2 mm to (217.6, 89.4), turned to 0 degrees
- moved J1 103.6 mm to (195.9, 55.2), turned to 0 degrees
- moved D6 98.8 mm to (222.8, 121.3), turned to 0 degrees
- moved R16 96.2 mm to (217.0, 95.4)
- moved D5 95.2 mm to (217.5, 73.0), turned to 0 degrees
- moved U7 93.3 mm to (62.2, 109.9), turned to 0 degrees
- moved C9 92.0 mm to (95.5, 152.2), turned to 90 degrees
- moved D4 91.8 mm to (217.3, 98.2), turned to 0 degrees
- moved R19 78.4 mm to (226.2, 119.0), turned to 0 degrees
- moved R17 73.8 mm to (226.2, 121.3)
- moved JP2 70.8 mm to (217.3, 82.2), turned to 0 degrees
- moved C16 64.9 mm to (180.6, 75.3), turned to 0 degrees
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Connections:
- C1 pad 1: +3V3 -> /CH340_XI
- C12 pad 1: Net-(#FLG05-pwr) -> Net-(U6-BOOT)
- C12 pad 2: GND -> /BST_SW
- C14 pad 1: +3V3 -> Net-(U6-FB)
- C14 pad 2: GND -> +5V
- C15 pad 1: +3V3 -> +5V
- C16 pad 1: +3V3 -> +5V
- C17 pad 1: +3V3 -> +5V
- C18 pad 1: +5V -> +3V3
- C19 pad 1: Net-(U9-COMP) -> Net-(U8-EN)
- C20 pad 1: Net-(C20-Pad1) -> +3V3
- C21 pad 1: Net-(U9-SS) -> /LED_VOUT
- C3 pad 1: +3V3 -> /CH340_XO
- C4 pad 1: /ESP32+CH340/CH340_XI -> +3V3
- C5 pad 1: /ESP32+CH340/CH340_XO -> Net-(U1-VCC)
- C7 pad 1: VIN -> +3V3
- C8 pad 1: +3V3 -> /VBUS_USBC
- C9 pad 1: VOUT_LED -> /VBUS_POSTFILTER
- D1 pad 2: /Power+USB/VBUS_USBC -> Net-(D1-A)
- D2 pad 1: GND -> +5V
- D2 pad 2: DAT2 -> /VBUS_FUSED
- D3 pad 1: +5V -> GND
- D4 pad 1: ESP32_TX -> GND
- D5 pad 1: ESP32_RX -> /LED_DAT2
- D5 pad 2: Net-(D5-A) -> /LED_DAT1
- D6 pad 1: GND -> /LED_DAT4
- D6 pad 2: Net-(D6-A) -> /LED_DAT3
- D7 pad 1: GND -> VIN
- D7 pad 2: DAT1 -> GND
- F1 pad 1: /Power+USB/VIN_RAW -> /VBUS_POSTFILTER
- F1 pad 2: /Power+USB/VIN_RPP -> /VBUS_FUSED
- FB1 pad 1: +5V -> /VBUS_USBC
- FB1 pad 2: Net-(#FLG05-pwr) -> /VBUS_POSTFILTER
- J1 pad A4: /Power+USB/VBUS_USBC -> /VBUS_USBC
- J1 pad A6: /Power+USB/D+ -> /DP
- J1 pad A7: /Power+USB/D- -> /DN
- J1 pad A9: /Power+USB/VBUS_USBC -> /VBUS_USBC
- J1 pad B4: /Power+USB/VBUS_USBC -> /VBUS_USBC
- J1 pad B6: /Power+USB/D+ -> /DP
- J1 pad B7: /Power+USB/D- -> /DN
- J1 pad B9: /Power+USB/VBUS_USBC -> /VBUS_USBC
- J1 pad S1: unconnected-(J1-SHIELD-PadS1) -> Net-(J1-SHIELD)
- J2 pad 1: /Power+USB/VIN_RAW -> /SCL
- J2 pad 2: GND -> /SDA
- J3 pad 1: /Power+USB/VBUS_MICROUSB -> /ESP32_TX
- J3 pad 2: unconnected-(J3-D--Pad2) -> /ESP32_RX
- J3 pad 3: unconnected-(J3-D+-Pad3) -> +3V3
- J3 pad 4: unconnected-(J3-ID-Pad4) -> GND
- J4 pad 1: GND -> /VIN_RAW
- J4 pad 2: +3V3 -> GND
- J4 pad 3: SDA -> /VIN_MINUS
- J5 pad 1: /Power+USB/VIN_RAW -> /VIN_MINUS
- J5 pad 2: GND -> /VIN_RAW
- JP1 pad 1: GND -> VIN
- JP2 pad 2: /Power+USB/INA180_IN -> /LED_VOUT
- K1 pad 1: /Power+USB/INA180_IN -> /LED_VOUT
- K1 pad 2: Net-(D3-A) -> Net-(D1-A)
- MK1 pad 1: SD -> /I2S_WS
- MK1 pad 2: +3V3 -> GND
- MK1 pad 4: GND -> /I2S_SCK
- MK1 pad 5: WS -> +3V3
- MK1 pad 6: SCK -> /I2S_SD
- Q1 pad 2: GND -> /nRTS
- Q1 pad 3: Net-(D3-A) -> EN
- Q2 pad 2: /ESP32+CH340/nRTS -> /nDTR
- Q2 pad 3: IO0 -> /IO0
- Q3 pad 2: /ESP32+CH340/nDTR -> GND
- Q3 pad 3: EN -> Net-(D1-A)
- R1 pad 1: Net-(J1-CC1) -> GND
- R1 pad 2: GND -> Net-(J1-SHIELD)
- R10 pad 1: IO0 -> /RELAY_CTRL
- R10 pad 2: Net-(BOOT1-Pad1) -> Net-(Q3-B)
- R11 pad 1: +3V3 -> Net-(U6-FB)
- R11 pad 2: Net-(D4-A) -> +5V
- R12 pad 1: +3V3 -> GND
- R12 pad 2: SW2 -> Net-(U6-FB)
- R13 pad 2: Net-(D5-A) -> /SDA
- R14 pad 1: /Power+USB/INA180_IN -> +3V3
- R14 pad 2: VOUT_LED -> /SCL
- R15 pad 2: SDA -> /IO0
- R16 pad 2: Net-(D6-A) -> /SW_L
- R17 pad 2: SW3 -> /SW_R
- R18 pad 1: RELAY_CTRL -> +3V3
- R18 pad 2: Net-(D9-A) -> Net-(D3-A)
- R19 pad 1: +3V3 -> /IO0
- R19 pad 2: SCL -> Net-(R19-Pad2)
- R2 pad 1: Net-(J1-CC2) -> +3V3
- R2 pad 2: GND -> /TEMP
- R20 pad 1: Net-(C20-Pad1) -> /RELAY_CTRL
- R20 pad 2: Net-(U9-COMP) -> Net-(D4-A)
- R3 pad 1: Net-(U1-TXD) -> Net-(J1-CC2)
- R3 pad 2: ESP32_RX -> GND
- R4 pad 1: Net-(U1-RXD) -> Net-(J1-CC1)
- R4 pad 2: ESP32_TX -> GND
- R5 pad 1: RELAY_CTRL -> +3V3
- R5 pad 2: Net-(Q1-B) -> Net-(U1-VCC)
- R6 pad 1: /ESP32+CH340/nDTR -> Net-(U3-TXD)
- R6 pad 2: Net-(Q2-B) -> /ESP32_RX
- R7 pad 1: /ESP32+CH340/nRTS -> Net-(U3-RXD)
- R7 pad 2: Net-(Q3-B) -> /ESP32_TX
- R8 pad 1: +3V3 -> /nDTR
- R8 pad 2: IO0 -> Net-(Q1-B)
- R9 pad 1: +3V3 -> /nRTS
- R9 pad 2: TEMP -> Net-(Q2-B)
- U1 pad 2: Net-(U1-TXD) -> Net-(U1-VCC)
- U1 pad 3: Net-(U1-RXD) -> /IR_CTRL
- U1 pad 4: +3V3 -> GND
- U2 pad 1: /Power+USB/D- -> GND
- U2 pad 2: GND -> /TEMP
- U2 pad 3: /Power+USB/D+ -> +3V3
- U3 pad 10: WS -> unconnected-(U3-~{DSR}-Pad10)
- U3 pad 13: unconnected-(U3-IO14-Pad13) -> /nDTR
- U3 pad 14: IR_CTRL -> /nRTS
- U3 pad 15: GND -> unconnected-(U3-R232-Pad15)
- U3 pad 16: RELAY_CTRL -> +3V3
- U3 pad 2: +3V3 -> Net-(U3-TXD)
- U3 pad 3: EN -> Net-(U3-RXD)
- U3 pad 4: unconnected-(U3-SENSOR_VP-Pad4) -> +3V3
- U3 pad 5: unconnected-(U3-SENSOR_VN-Pad5) -> /USB_DP
- U3 pad 6: V_SENSE -> /USB_DN
- U3 pad 7: unconnected-(U3-IO35-Pad7) -> /CH340_XI
- U3 pad 8: SD -> /CH340_XO
- U3 pad 9: SCK -> unconnected-(U3-~{CTS}-Pad9)
- U4 pad 1: IR_CTRL -> /DP
- U4 pad 3: +3V3 -> /DN
- U6 pad 1: Net-(#FLG05-pwr) -> GND
- U6 pad 2: GND -> /BST_SW
- U6 pad 3: Net-(#FLG05-pwr) -> VIN
- U6 pad 4: unconnected-(U6-NC-Pad4) -> Net-(U6-FB)
- U6 pad 5: +3V3 -> Net-(JP1-B)
- U7 pad 2: TEMP -> /LED_DAT1_3V3
- U7 pad 3: +3V3 -> /LED_DAT1
- U8 pad 1: unconnected-(U8-1OE-Pad1) -> Net-(U8-EN)
- U8 pad 2: CLK2_3V3 -> GND
- U8 pad 3: unconnected-(U8-2Y0-Pad3) -> Net-(U8-EN)
- U8 pad 4: DAT2_3V3 -> unconnected-(U8-NC-Pad4)
- U8 pad 5: unconnected-(U8-2Y1-Pad5) -> +3V3
- Y1 pad 1: /ESP32+CH340/CH340_XI -> /CH340_XI
- Y1 pad 3: /ESP32+CH340/CH340_XO -> /CH340_XO
Routing:
- net GND: track 117.7 -> 0.00 mm, vias 36 -> 0
- net ESP32_TX: track 76.7 -> 0.00 mm, vias 3 -> 0
- net ESP32_RX: track 70.0 -> 0.00 mm, vias 3 -> 0
- net RELAY_CTRL: track 62.0 -> 0.00 mm
- net +3V3: track 50.1 -> 0.00 mm, vias 13 -> 0
- net IR_CTRL: track 41.7 -> 0.00 mm
- net V_SENSE: track 40.6 -> 0.00 mm
- net +5V: track 37.7 -> 0.00 mm, vias 5 -> 0
- net SW2: track 31.4 -> 0.00 mm, vias 1 -> 0
- net DAT1: track 30.3 -> 0.00 mm
- net IO0: track 29.2 -> 0.00 mm, vias 2 -> 0
- net CLK1: track 26.8 -> 0.00 mm
- net Net-(BOOT1-Pad1): track 22.7 -> 0.00 mm, vias 3 -> 0
- net SD: track 22.5 -> 0.00 mm, vias 1 -> 0
- net SW3: track 21.7 -> 0.00 mm, vias 1 -> 0
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- added copper zone on B.Cu, net +3V3
- added copper zone on F.Cu, net +5V
- added copper zone on F.Cu, net /BST_SW
- added copper zone on F.Cu, net /LED_VOUT
- added copper zone on F.Cu, net /VBUS_FUSED
- added copper zone on F.Cu, net /VBUS_POSTFILTER
- added copper zone on B.Cu, net /VBUS_USBC
- added copper zone on F.Cu, net GND
- added copper zone on In2.Cu, net GND
- removed copper zone on In2.Cu, net +3V3
- removed copper zone on In2.Cu, net +5V
- removed copper zone on F.Cu, net /Power+USB/INA180_IN
- removed copper zone on In2.Cu, net /Power+USB/VBUS_USBC
- removed copper zone on F.Cu, net /Power+USB/VIN_RAW
- removed copper zone on F.Cu, net /Power+USB/VIN_RPP
- removed copper zone on F.Cu, net VIN
- removed copper zone on F.Cu, net VOUT_LED
Other:
- board size 94.6 x 64.6 mm -> 95 x 65 mm
- board text removed: "5-24VDC - +"
- board text removed: "BUCK DISBABLE"
- board text removed: "Button 1"
- board text removed: "Button 2"
- board text removed: "Button 3"
- board text removed: "CLK2 DAT2"
- board text removed: "GND CLK1 DAT1 VCC"
- board text removed: "GND TX RX"
- board text removed: "JLCJLCJLCJLC"
- board text removed: "LuminX WLED"
- board text removed: "Michael Gross"
- board text removed: "POWER"
- board text removed: "RELAY"
- board text removed: "RELAY DISABLE"
- board text removed: "RX"
- board text removed: "TX"
- board text removed: "VIN = 5V INT 5V (max 3A)"
- board text removed: "v1.0 - 03.2023"

Commit message: Add backups
Parts:
- removed C1, C3: 30p, Capacitor_SMD:C_0603_1608Metric
- removed C11: 10u, Capacitor_SMD:C_1206_3216Metric
- removed C12: 100n, Capacitor_SMD:C_0603_1608Metric
- removed C14: 47p, Capacitor_SMD:C_0603_1608Metric
- removed C15, C16: 22u, Capacitor_SMD:C_1206_3216Metric
- removed D2: SS34, Diode_SMD:D_SMA
- removed D5: SP0502BAHT, Package_TO_SOT_SMD:SOT-23
- removed F3: Fuse, Fuse:Fuseholder_Clip-5x20mm_Littelfuse_521_Lateral_P17.00x5.00mm_D1.30mm_Horizontal
- removed H5, H6, H7, H8: MountingHole, MountingHole:MountingHole_3.2mm_M3_Pad_Via
- removed JP1: Jumper_2_Open, Connector_PinHeader_2.54mm:PinHeader_1x02_P2.54mm_Vertical
- removed L1: 10u/2A, Inductor_SMD:L_Sunlord_MWSA0603S
- removed MK1: MIC_I2S_INMP441, MG_Footprint_Lib:MIC_I2S_ICS-43434+INMP441
- removed R12: 13k7, Resistor_SMD:R_0603_1608Metric
- removed SW_C1, SW_L1, SW_R1: SW_Push, Button_Switch_SMD:SW_SPST_PTS645
- removed U6: TPS54302, Package_TO_SOT_SMD:SOT-23-6
- removed Y1: 12MHz, Crystal:Crystal_SMD_3225-4Pin_3.2x2.5mm
- added C22: 10u, Capacitor_SMD:C_1206_3216Metric, F.Cu at (112.3, 146.6)
- added C23: 100n, Capacitor_SMD:C_0603_1608Metric, F.Cu at (113.1, 138.3)
- added C24: 47p, Capacitor_SMD:C_0603_1608Metric, F.Cu at (108.0, 140.8)
- added C25: 22u, Capacitor_SMD:C_1206_3216Metric, F.Cu at (117.1, 146.6)
- added C26: 22u, Capacitor_SMD:C_1206_3216Metric, F.Cu at (117.1, 144.2)
- added F4: 3.5A, MG_Footprint_Lib:Fuseholder_Clip-5x20mm_Littelfuse_521_Lateral_P17.00x5.00mm_D1.30mm_Horizontal, F.Cu at (178.0, 116.7)
- added L2: MWSA0603S-6R8MT, Inductor_SMD:L_Sunlord_MWSA0603S, F.Cu at (119.3, 139.2)
- added MK2: ICS-43434, Sensor_Audio:InvenSense_ICS-43434-6_3.5x2.65mm, F.Cu at (178.9, 74.6)
- added Q4: AO3401A, Package_TO_SOT_SMD:SOT-23, F.Cu at (197.4, 72.1)
- added R21: 158k, Resistor_SMD:R_0603_1608Metric, F.Cu at (109.5, 140.8)
- added R22: 30k1, Resistor_SMD:R_0603_1608Metric, F.Cu at (110.1, 138.3)
- added SW1: SW_Push, Button_Switch_SMD:SW_SPST_PTS645, B.Cu at (163.6, 98.3)
- added SW2: SW_Push, Button_Switch_SMD:SW_SPST_PTS645, B.Cu at (148.6, 98.3)
- added SW3: SW_Push, Button_Switch_SMD:SW_SPST_PTS645, B.Cu at (133.6, 98.3)
- added U9: TSOP382xx, OptoDevice:Vishay_MINICAST-3Pin, F.Cu at (137.3, 89.2)
- C4: moved to F.Cu
- D6: value SP0502BAHT -> SS34; footprint Package_TO_SOT_SMD:SOT-23 -> Diode_SMD:D_SMA
- F1: footprint Fuse:Fuse_1206_3216Metric -> MG_Footprint_Lib:Fuseholder_Clip-5x20mm_Littelfuse_521_Lateral_P17.00x5.00mm_D1.30mm_Horizontal
- FB1: value 120R -> 100R 3A
- J2, J3: value JST PH -> JST SH; footprint Connector_JST:JST_PH_B4B-PH-SM4-TB_1x04-1MP_P2.00mm_Vertical -> Connector_JST:JST_SH_BM04B-SRSS-TB_1x04-1MP_P1.00mm_Vertical
- R11: value 100k -> 10k; footprint Resistor_SMD:R_0603_1608Metric -> Resistor_SMD:R_0805_2012Metric
- U1: value ~ -> CH340C; footprint MG_Footprint_Lib:Vishay_IR_Heimdall -> Package_SO:SOIC-16_3.9x9.9mm_P1.27mm
- U3: value CH340G -> ESP32-WROOM-32E; footprint Package_SO:SOIC-16_3.9x9.9mm_P1.27mm -> RF_Module:ESP32-WROOM-32D
- U4: value USBLC6-2P6 -> AP63300; footprint Package_TO_SOT_SMD:SOT-666 -> Package_TO_SOT_SMD:TSOT-23-6
- U5: value ESP32-WROOM-32D -> USBLC6-2SC6; footprint RF_Module:ESP32-WROOM-32D -> Package_TO_SOT_SMD:SOT-23-6
- moved U7 112.9 mm to (172.8, 87.3)
- moved J2 111.7 mm to (209.8, 49.5), turned to 0 degrees
- moved Q2 100.5 mm to (234.6, 94.8)
- moved Q3 100.5 mm to (234.6, 91.3)
- moved J1 90.8 mm to (110.1, 84.8), turned to -90 degrees
- moved R13 84.1 mm to (72.6, 87.0)
- moved R18 84.1 mm to (60.4, 88.8)
- moved R9 81.2 mm to (80.7, 63.3)
- moved J6 80.5 mm to (186.0, 115.8), turned to 90 degrees
- moved R11 78.8 mm to (202.1, 71.2)
- moved C9 76.1 mm to (119.1, 79.8)
- moved J4 72.1 mm to (119.6, 110.5), turned to -90 degrees
- moved C10 68.6 mm to (117.6, 73.8), turned to 180 degrees
- moved C21 67.3 mm to (173.7, 106.2), turned to 90 degrees
- moved R3 61.7 mm to (116.6, 87.3), turned to 0 degrees
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Connections:
- C10 pad 1: /VBUS_POSTFILTER -> /VBUS
- C19 pad 1: Net-(U8-EN) -> +5V
- C20 pad 1: +3V3 -> Net-(U8-VOUT)
- C5 pad 1: Net-(U1-VCC) -> Net-(U9-Vs)
- C8 pad 1: /VBUS_USBC -> /VBUS_RAW
- C9 pad 1: /VBUS_POSTFILTER -> /VBUS
- D6 pad 1: /LED_DAT4 -> +5V
- D6 pad 2: /LED_DAT3 -> /BUCK_5V
- D7 pad 1: VIN -> unconnected-(D7-K-Pad1)
- F1 pad 1: /VBUS_POSTFILTER -> /LED_VOUT
- F1 pad 2: /VBUS_FUSED -> Net-(J6-Pin_1)
- F2 pad 1: +5V -> Net-(U8-VOUT)
- F2 pad 2: Net-(U8-EN) -> +3V3
- FB1 pad 1: /VBUS_USBC -> /VBUS_RAW
- FB1 pad 2: /VBUS_POSTFILTER -> /VBUS
- J1 pad A4: /VBUS_USBC -> /VBUS_RAW
- J1 pad A9: /VBUS_USBC -> /VBUS_RAW
- J1 pad B4: /VBUS_USBC -> /VBUS_RAW
- J1 pad B9: /VBUS_USBC -> /VBUS_RAW
- J4 pad 1: /VIN_RAW -> VIN
- J5 pad 2: /VIN_RAW -> VIN
- J6 pad 1: /LED_VOUT -> Net-(J6-Pin_1)
- J6 pad 5: /LED_VOUT -> Net-(J6-Pin_5)
- R11 pad 1: Net-(U6-FB) -> /BUCK_5V
- R11 pad 2: +5V -> GND
- R16 pad 2: /SW_L -> /SW2
- R17 pad 2: /SW_R -> /SW3
- R5 pad 2: Net-(U1-VCC) -> Net-(U9-Vs)
- R6 pad 1: Net-(U3-TXD) -> Net-(U1-TXD)
- R7 pad 1: Net-(U3-RXD) -> Net-(U1-RXD)
- U1 pad 2: Net-(U1-VCC) -> Net-(U1-TXD)
- U1 pad 3: /IR_CTRL -> Net-(U1-RXD)
- U1 pad 4: GND -> +3V3
- U3 pad 10: unconnected-(U3-~{DSR}-Pad10) -> /I2S_WS
- U3 pad 13: /nDTR -> unconnected-(U3-IO14-Pad13)
- U3 pad 14: /nRTS -> /IR_CTRL
- U3 pad 15: unconnected-(U3-R232-Pad15) -> GND
- U3 pad 16: +3V3 -> /RELAY_CTRL
- U3 pad 2: Net-(U3-TXD) -> +3V3
- U3 pad 3: Net-(U3-RXD) -> EN
- U3 pad 4: +3V3 -> unconnected-(U3-SENSOR_VP-Pad4)
- U3 pad 5: /USB_DP -> unconnected-(U3-SENSOR_VN-Pad5)
- U3 pad 6: /USB_DN -> /V_SENSE
- U3 pad 7: /CH340_XI -> unconnected-(U3-IO35-Pad7)
- U3 pad 8: /CH340_XO -> /I2S_SD
- U3 pad 9: unconnected-(U3-~{CTS}-Pad9) -> /I2S_SCK
- U4 pad 1: /DP -> Net-(U4-FB)
- U4 pad 2: GND -> VIN
- U4 pad 3: /DN -> VIN
- U4 pad 4: /USB_DN -> GND
- U4 pad 5: /VBUS_USBC -> /BUCK_SW
- U4 pad 6: /USB_DP -> Net-(U4-BST)
- U5 pad 1: GND -> /DP
- U5 pad 2: +3V3 -> GND
- U5 pad 3: EN -> /DN
- U5 pad 4: unconnected-(U5-SENSOR_VP-Pad4) -> /USB_DN
- U5 pad 5: unconnected-(U5-SENSOR_VN-Pad5) -> /VBUS_RAW
- U5 pad 6: /V_SENSE -> /USB_DP
- U8 pad 1: Net-(U8-EN) -> +5V
- U8 pad 3: Net-(U8-EN) -> +5V
- U8 pad 5: +3V3 -> Net-(U8-VOUT)
Routing:
- removed copper zone on B.Cu, net +3V3
- removed copper zone on F.Cu, net +5V
- removed copper zone on F.Cu, net /BST_SW
- removed copper zone on F.Cu, net /LED_VOUT
- removed copper zone on F.Cu, net /VBUS_FUSED
- removed copper zone on F.Cu, net /VBUS_POSTFILTER
- removed copper zone on B.Cu, net /VBUS_USBC
- removed copper zone on F.Cu, net GND
- removed copper zone on In1.Cu, net GND
- removed copper zone on In2.Cu, net GND
Other:
- board size 95 x 65 mm -> 85 x 55 mm
