File: Hardware/LuminX Pro.kicad_sch (KiCad schematic)
At the start: 4 parts

Commit message: Revise v2 schematic
Parts:
- added C1, C3: 30p, Capacitor_SMD:C_0603_1608Metric, symbol Device:C_Small
- added C10: 10u, Capacitor_SMD:C_1206_3216Metric, symbol MG_Symbol_Lib:CAP_1206
- added C11: 10u, Capacitor_SMD:C_1206_3216Metric, symbol Device:C_Small
- added C12, C17, C18, C2, C4, C6: 100n, Capacitor_SMD:C_0603_1608Metric, symbol Device:C_Small
- added C13: 10u, Capacitor_SMD:C_0805_2012Metric, symbol Device:C_Small
- added C14: 47p, Capacitor_SMD:C_0603_1608Metric, symbol Device:C_Small
- added C15, C16: 22u, Capacitor_SMD:C_1206_3216Metric, symbol Device:C_Small
- added C19, C20: 1u, Capacitor_SMD:C_0603_1608Metric, symbol Device:C_Small
- added C21: 1000u, Capacitor_THT:CP_Radial_D12.5mm_P5.00mm, symbol Device:C_Polarized_Small
- added C5: 2u2, Capacitor_SMD:C_0805_2012Metric, symbol MG_Symbol_Lib:CAP_0805
- added C7: 10u, Capacitor_SMD:C_0805_2012Metric, symbol Device:C_Polarized_Small
- added C8: 10n, Capacitor_SMD:C_0603_1608Metric, symbol MG_Symbol_Lib:CAP_0603
- added C9: 100n, Capacitor_SMD:C_0603_1608Metric, symbol MG_Symbol_Lib:CAP_0603
- added D1, D7: US1G, Diode_SMD:D_SMA, symbol Diode:US1G
- added D2: SS34, Diode_SMD:D_SMA, symbol Diode:1N5820
- added D3: GREEN, LED_SMD:LED_0805_2012Metric, symbol Device:LED
- added D4: AMBER, LED_SMD:LED_0805_2012Metric, symbol Device:LED
- added D5, D6: SP0502BAHT, Package_TO_SOT_SMD:SOT-23, symbol Power_Protection:SP0502BAHT
- added F1: 3.5A, Fuse:Fuse_1206_3216Metric, symbol Device:Polyfuse
- added F2: 750mA, Fuse:Fuse_1206_3216Metric, symbol Device:Polyfuse_Small
- added F3: Fuse, Fuse:Fuseholder_Clip-5x20mm_Littelfuse_521_Lateral_P17.00x5.00mm_D1.30mm_Horizontal, symbol Device:Fuse
- added FB1: 120R, Inductor_SMD:L_0603_1608Metric, symbol Device:FerriteBead_Small
- added H5, H6, H7, H8: MountingHole, MountingHole:MountingHole_3.2mm_M3_Pad_Via, symbol Mechanical:MountingHole_Pad
- added J1: GCT USB4105, Connector_USB:USB_C_Receptacle_GCT_USB4105-xx-A_16P_TopMnt_Horizontal, symbol MG_Symbol_Lib:Conn_USB_C_USB2.0_GCT_USB4105
- added J2, J3: JST PH, Connector_JST:JST_PH_B4B-PH-SM4-TB_1x04-1MP_P2.00mm_Vertical, symbol Connector_Generic:Conn_01x04
- added J4: GCT DCJ200-10, MG_Footprint_Lib:Conn_BarrelJack_GCT_DCJ200-10-A_Horizontal, symbol MG_Symbol_Lib:Conn_BarrelJack_GCT_DCJ200-10-A_Horizontal
- added J5: 5mm Screw Terminal, TerminalBlock_Phoenix:TerminalBlock_Phoenix_MKDS-1,5-2_1x02_P5.00mm_Horizontal, symbol Connector:Screw_Terminal_01x02
- added J6: Phoenix MKDS x8 5mm, TerminalBlock_Phoenix:TerminalBlock_Phoenix_MKDS-1,5-8_1x08_P5.00mm_Horizontal, symbol Connector:Screw_Terminal_01x08
- added JP1, JP2, JP3: Jumper_2_Open, Connector_PinHeader_2.54mm:PinHeader_1x02_P2.54mm_Vertical, symbol Jumper:Jumper_2_Open
- added K1: G5LE-1, Relay_THT:Relay_SPDT_Omron-G5LE-1, symbol Relay:G5LE-1
- added L1: 10u/2A, Inductor_SMD:L_Sunlord_MWSA0603S, symbol Device:L
- added MK1: MIC_I2S_INMP441, MG_Footprint_Lib:MIC_I2S_ICS-43434+INMP441, symbol MG_Symbol_Lib:MIC_I2S_INMP441
- added Q1, Q2, Q3: BC847, Package_TO_SOT_SMD:SOT-23, symbol Transistor_BJT:BC847
- added R1: 0R, Resistor_SMD:R_0603_1608Metric, symbol Device:R_Small
- added R10, R5: 220R, Resistor_SMD:R_0603_1608Metric, symbol Device:R_Small
- added R11: 100k, Resistor_SMD:R_0603_1608Metric, symbol Device:R_Small
- added R12: 13k7, Resistor_SMD:R_0603_1608Metric, symbol Device:R_Small
- added R13, R14: 4k7, Resistor_SMD:R_0603_1608Metric, symbol Device:R_Small
- added R15, R16, R17, R2, R8, R9: 10k, Resistor_SMD:R_0603_1608Metric, symbol Device:R_Small
- added R18, R20: 1k, Resistor_SMD:R_0603_1608Metric, symbol Device:R_Small
- added R19, R6, R7: 470R, Resistor_SMD:R_0603_1608Metric, symbol Device:R_Small
- added R3, R4: 5k1, Resistor_SMD:R_0603_1608Metric, symbol Device:R_Small
- added SW_C1, SW_L1, SW_R1: SW_Push, Button_Switch_SMD:SW_SPST_PTS645, symbol Switch:SW_Push
- added U1: ~, MG_Footprint_Lib:Vishay_IR_Heimdall, symbol MG_Symbol_Lib:IR_Receiver_TSOP75438
- added U2: DS18B20, Package_TO_SOT_THT:TO-92_Inline, symbol Sensor_Temperature:DS18B20
- added U3: CH340G, Package_SO:SOIC-16_3.9x9.9mm_P1.27mm, symbol Interface_USB:CH340G
- added U4: USBLC6-2P6, Package_TO_SOT_SMD:SOT-666, symbol Power_Protection:USBLC6-2P6
- added U5: ESP32-WROOM-32D, RF_Module:ESP32-WROOM-32D, symbol RF_Module:ESP32-WROOM-32D
- added U6: TPS54302, Package_TO_SOT_SMD:SOT-23-6, symbol Regulator_Switching:TPS54302
- added U7: 74AHCT125, Package_SO:SO-14_3.9x8.65mm_P1.27mm, symbol MG_Symbol_Lib:74AHC125
- added U8: AP2112K-3.3, Package_TO_SOT_SMD:SOT-23-5, symbol Regulator_Linear:AP2112K-3.3
- added Y1: 12MHz, Crystal:Crystal_SMD_3225-4Pin_3.2x2.5mm, symbol Device:Crystal_GND24
Connections:
- net GND: now also C1.2, C10.2, C11.2, C13.2, C15.2, C16.2, C17.2, C18.2, C19.2, C2.2, C20.2, C21.2, C3.2, C4.2, C5.2, C6.2, C7.2, C8.2, C9.2, D3.1 (K), D4.1 (K), D5.3 (A), D6.3 (A), D7.2 (A), H5.1, H6.1, H7.1, H8.1, J1.A1 (GND), J1.A12 (GND), J1.B1 (GND), J1.B12 (GND), J2.4 (Pin_4), J3.4 (Pin_4), J4.2, J6.4 (Pin_4), J6.8 (Pin_8), MK1.2 (L/R), MK1.3 (GND), Q3.2 (E), R1.1, R12.1, R3.2, R4.2, SW_C1.2, SW_L1.2, SW_R1.2, U1.1 (GND), U1.4 (GND), U2.1 (GND), U3.1 (GND), U4.2 (GND), U5.1 (GND), U5.15 (GND), U5.38 (GND), U5.39 (GND), U6.1 (GND), U7.1 (1OE), U7.10 (3OE), U7.13 (4OE), U7.4 (2OE), U7.7 (GND), U8.2 (GND), Y1.2, Y1.4
- new net: J1.B5 (CC2), R3.1
- new net: Q3.1 (B), R10.2
- new net: C14.1, R11.1, R12.2, U6.4 (FB)
- new net: R19.2, SW_C1.1
- new net: D4.2 (A), R20.2
- new net: C5.1, R5.2, U1.2 (VCC)
- new net: J1.S1 (SHIELD), R1.2
- new net: JP1.2 (B), U6.5 (EN)
- new net: C12.1, U6.6 (BOOT)
- new net: D1.2 (A), K1.2, Q3.3 (C)
- new net: R6.1, U3.2 (TXD)
- new net: C19.1, F2.2, U8.1 (VIN), U8.3 (EN)
- new net: J1.A5 (CC1), R4.1
- new net: Q1.1 (B), R8.2
- new net: D3.2 (A), R18.2
- new net: Q2.1 (B), R9.2
- new net: R7.1, U3.3 (RXD)
- new net +3V3: C13.1, C18.1, C2.1, C20.1, C4.1, C6.1, C7.1, J2.3 (Pin_3), J3.3 (Pin_3), MK1.5 (VDD), R13.1, R14.1, R15.1, R16.1, R17.1, R18.1, R2.1, R5.1, U2.3 (V_{DD}), U3.16 (VCC), U3.4 (V3), U5.2 (VDD), U8.5 (VOUT)
- new net +5V: C14.2, C15.1, C16.1, C17.1, D1.1 (K), D2.1 (K), F2.1, JP3.2 (B), K1.5, L1.2, R11.2, U7.14 (VCC)
- new net BST_SW: C12.2, L1.1, U6.2 (SW)
- new net CH340_XI: C1.1, U3.7 (XI), Y1.1
- new net CH340_XO: C3.1, U3.8 (XO), Y1.3
- new net DN: J1.A7 (D-), J1.B7 (D-), U4.3 (I/O2)
- new net DP: J1.A6 (D+), J1.B6 (D+), U4.1 (I/O1)
- new net EN: Q1.3 (C), U5.3 (EN)
- new net ESP32_RX: J3.2 (Pin_2), R6.2, U5.34 (RXD0/IO3)
- new net ESP32_TX: J3.1 (Pin_1), R7.2, U5.35 (TXD0/IO1)
- new net I2S_SCK: MK1.4 (SCK), U5.9 (IO33)
- new net I2S_SD: MK1.6 (SD), U5.8 (IO32)
- new net I2S_WS: MK1.1 (WS), U5.10 (IO25)
- new net IO0: Q2.3 (C), R15.2, R19.1, U5.25 (IO0)
- new net IR_CTRL: U1.3 (OUT), U5.14 (IO12)
- new net LED_DAT1: D5.2 (K), J6.2 (Pin_2), U7.3 (1Y)
- new net LED_DAT1_3V3: U5.24 (IO2), U7.2 (1A)
- new net LED_DAT2: D5.1 (K), J6.3 (Pin_3), U7.6 (2Y)
- new net LED_DAT2_3V3: U5.29 (IO5), U7.5 (2A)
- new net LED_DAT3: D6.2 (K), J6.6 (Pin_6), U7.8 (3Y)
- new net LED_DAT3_3V3: U5.30 (IO18), U7.9 (3A)
- new net LED_DAT4: D6.1 (K), J6.7 (Pin_7), U7.11 (4Y)
- new net LED_DAT4_3V3: U5.31 (IO19), U7.12 (4A)
- new net LED_VOUT: C21.1, J6.1 (Pin_1), J6.5 (Pin_5), JP2.2 (B), K1.1
- new net RELAY_CTRL: R10.1, R20.1, U5.16 (IO13)
- new net SCL: J2.1 (Pin_1), R14.2, U5.36 (IO22)
- new net SDA: J2.2 (Pin_2), R13.2, U5.33 (IO21)
- new net SW2: U5.26 (IO4)
- new net SW3: U5.27 (IO16)
- new net SW_L: R16.2, SW_L1.1
- new net SW_R: R17.2, SW_R1.1
- new net TEMP: R2.2, U2.2 (DQ), U5.23 (IO15)
- new net USB_DN: U3.6 (UD-), U4.4 (I/O2)
- new net USB_DP: U3.5 (UD+), U4.6 (I/O1)
- new net VBUS_FUSED: D2.2 (A), F1.2
- new net VBUS_POSTFILTER: C10.1, C9.1, F1.1, FB1.2
- new net VBUS_USBC: C8.1, FB1.1, J1.A4 (VBUS), J1.A9 (VBUS), J1.B4 (VBUS), J1.B9 (VBUS), U4.5 (VBUS)
- new net VIN: C11.1, D7.1 (K), F3.2, JP1.1 (A), JP2.1 (A), JP3.1 (A), K1.3, U6.3 (VIN)
- new net VIN_MINUS: J4.3, J5.1 (Pin_1)
- new net VIN_RAW: F3.1, J4.1, J5.2 (Pin_2)
- new net V_SENSE: U5.6 (IO34)
- new net nDTR: Q2.2 (E), R8.1, U3.13 (~{DTR})
- new net nRTS: Q1.2 (E), R9.1, U3.14 (~{RTS})
- no-connect marks 0 -> 22
Other:
- removed sheet ESP32+CH340
- removed sheet Power+USB
- note added: "2.1mm Barrel Jack, Screw Terminal"
- note added: "3.3V LDO"
- note added: "5V Buck Converter"
- note added: "Boot Mode Selection"
- note added: "Buck Enable"
- note added: "Bypass Relay (max 3A)"
- note added: "CH340C/E USB to Serial"
- note added: "C_l = 2 * (C_load - C_stray)"
- note added: "C_stray = 3-5 pF"
- note added: "ESP-WROOM-32UE SoM"
- note added: "I2C & Serial Connectors"
- note added: "ICS43434 or INMP441 I2S Microphone"
- note added: "IR Receiver"
- note added: "In case CH340C is used leave C1, C2, Y1 unpopulated"
- note added: "LEDs"
- note added: "Level Shifter"
- note added: "Microphone"
- note added: "Power"
- note added: "Power Relay"
- note added: "Push Buttons"
- note added: "Temp Sensor"
- note added: "USB C Receptacle (power and data)"
- note added: "VIN = 5V"
- note added: "WS2812 Data Output"
- title: LuminX WLED -> LuminX Pro

Commit message: Add backups
Parts:
- removed C1, C3: 30p, Capacitor_SMD:C_0603_1608Metric, symbol Device:C_Small
- removed C11: 10u, Capacitor_SMD:C_1206_3216Metric, symbol Device:C_Small
- removed C12: 100n, Capacitor_SMD:C_0603_1608Metric, symbol Device:C_Small
- removed C14: 47p, Capacitor_SMD:C_0603_1608Metric, symbol Device:C_Small
- removed C15, C16: 22u, Capacitor_SMD:C_1206_3216Metric, symbol Device:C_Small
- removed D2: SS34, Diode_SMD:D_SMA, symbol Diode:1N5820
- removed D5, D6: SP0502BAHT, Package_TO_SOT_SMD:SOT-23, symbol Power_Protection:SP0502BAHT
- removed F3: Fuse, Fuse:Fuseholder_Clip-5x20mm_Littelfuse_521_Lateral_P17.00x5.00mm_D1.30mm_Horizontal, symbol Device:Fuse
- removed H5, H6, H7, H8: MountingHole, MountingHole:MountingHole_3.2mm_M3_Pad_Via, symbol Mechanical:MountingHole_Pad
- removed JP1: Jumper_2_Open, Connector_PinHeader_2.54mm:PinHeader_1x02_P2.54mm_Vertical, symbol Jumper:Jumper_2_Open
- removed L1: 10u/2A, Inductor_SMD:L_Sunlord_MWSA0603S, symbol Device:L
- removed MK1: MIC_I2S_INMP441, MG_Footprint_Lib:MIC_I2S_ICS-43434+INMP441, symbol MG_Symbol_Lib:MIC_I2S_INMP441
- removed R11: 100k, Resistor_SMD:R_0603_1608Metric, symbol Device:R_Small
- removed R12: 13k7, Resistor_SMD:R_0603_1608Metric, symbol Device:R_Small
- removed U1: ~, MG_Footprint_Lib:Vishay_IR_Heimdall, symbol MG_Symbol_Lib:IR_Receiver_TSOP75438
- removed U3: CH340G, Package_SO:SOIC-16_3.9x9.9mm_P1.27mm, symbol Interface_USB:CH340G
- removed U4: USBLC6-2P6, Package_TO_SOT_SMD:SOT-666, symbol Power_Protection:USBLC6-2P6
- removed U5: ESP32-WROOM-32D, RF_Module:ESP32-WROOM-32D, symbol RF_Module:ESP32-WROOM-32D
- removed U6: TPS54302, Package_TO_SOT_SMD:SOT-23-6, symbol Regulator_Switching:TPS54302
- removed Y1: 12MHz, Crystal:Crystal_SMD_3225-4Pin_3.2x2.5mm, symbol Device:Crystal_GND24
- added C22: 10u, Capacitor_SMD:C_1206_3216Metric, symbol Device:C_Small
- added C23: 100n, Capacitor_SMD:C_0603_1608Metric, symbol Device:C_Small
- added C24: 47p, Capacitor_SMD:C_0603_1608Metric, symbol Device:C_Small
- added C25, C26: 22u, Capacitor_SMD:C_1206_3216Metric, symbol Device:C_Small
- added D6: SS34, Diode_SMD:D_SMA, symbol Diode:SS34
- added F4: 3.5A, MG_Footprint_Lib:Fuseholder_Clip-5x20mm_Littelfuse_521_Lateral_P17.00x5.00mm_D1.30mm_Horizontal, symbol Device:Polyfuse
- added L2: MWSA0603S-6R8MT, Inductor_SMD:L_Sunlord_MWSA0603S, symbol Device:L
- added MK2: ICS-43434, Sensor_Audio:InvenSense_ICS-43434-6_3.5x2.65mm, symbol Sensor_Audio:ICS-43434
- added Q4: AO3401A, Package_TO_SOT_SMD:SOT-23, symbol Transistor_FET:AO3401A
- added R11: 10k, Resistor_SMD:R_0805_2012Metric, symbol Custom:R_0805
- added R21: 158k, Resistor_SMD:R_0603_1608Metric, symbol Device:R_Small
- added R22: 30k1, Resistor_SMD:R_0603_1608Metric, symbol Device:R_Small
- added TP1, TP2, TP3: TestPoint, symbol Connector:TestPoint
- added U1: CH340C, Package_SO:SOIC-16_3.9x9.9mm_P1.27mm, symbol Interface_USB:CH340C
- added U3: ESP32-WROOM-32E, RF_Module:ESP32-WROOM-32D, symbol RF_Module:ESP32-WROOM-32E
- added U4: AP63300, Package_TO_SOT_SMD:TSOT-23-6, symbol Regulator_Switching:AP63200WU
- added U5: USBLC6-2SC6, Package_TO_SOT_SMD:SOT-23-6, symbol Power_Protection:USBLC6-2SC6
- added U9: TSOP382xx, OptoDevice:Vishay_MINICAST-3Pin, symbol Interface_Optical:TSOP382xx
- F1: footprint Fuse:Fuse_1206_3216Metric -> MG_Footprint_Lib:Fuseholder_Clip-5x20mm_Littelfuse_521_Lateral_P17.00x5.00mm_D1.30mm_Horizontal
- FB1: value 120R -> 100R 3A
- J2, J3: value JST PH -> JST SH; footprint Connector_JST:JST_PH_B4B-PH-SM4-TB_1x04-1MP_P2.00mm_Vertical -> Connector_JST:JST_SH_BM04B-SRSS-TB_1x04-1MP_P1.00mm_Vertical
- R15: now not fitted
- renumbered SW_C1 to SW1, SW_L1 to SW2, SW_R1 to SW3
Connections:
- net SW_L is gone; now on net SW2: R16.2, SW2.1
- net SW_R is gone; now on net SW3: R17.2, SW3.1
- net +3V3: now also F2.2, MK2.5 (VDD), U1.16 (VCC), U1.4 (V3), U3.2 (VDD); no longer C20.1, U8.5 (VOUT)
- net +5V: now also C19.1, U8.1 (VIN), U8.3 (EN), D6.1 (K), Q4.2 (S); no longer F2.1
- net DN: now also U5.3 (I/O2)
- net DP: now also U5.1 (I/O1)
- net EN: now also U3.3 (EN)
- net ESP32_RX: now also U3.34 (RXD0/IO3)
- net ESP32_TX: now also U3.35 (TXD0/IO1)
- net GND: now also C22.2, C25.2, C26.2, MK2.2 (LR), MK2.3 (GND), R11.2, R22.1, TP2.1, U1.1 (GND), U3.1 (GND), U3.15 (GND), U3.38 (GND), U3.39 (GND), U4.4 (GND), U5.2 (GND), U9.2 (GND)
- net I2S_SCK: now also MK2.4 (SCK), U3.9 (IO33)
- net I2S_SD: now also MK2.6 (SD), U3.8 (IO32)
- net I2S_WS: now also MK2.1 (WS), U3.10 (IO25)
- net IO0: now also U3.25 (IO0)
- net IR_CTRL: now also U3.14 (IO12), U9.1 (OUT)
- net LED_DAT1_3V3: now also U3.24 (IO2)
- net LED_DAT2_3V3: now also U3.29 (IO5)
- net LED_DAT3_3V3: now also U3.30 (IO18)
- net LED_DAT4_3V3: now also U3.31 (IO19)
- net LED_VOUT: now also F1.1, F4.1; no longer J6.1 (Pin_1), J6.5 (Pin_5)
- net RELAY_CTRL: now also U3.16 (IO13)
- net SCL: now also U3.36 (IO22)
- net SDA: now also U3.33 (IO21)
- net SW2: now also U3.26 (IO4)
- net SW3: now also U3.27 (IO16)
- net TEMP: now also U3.23 (IO15)
- net USB_DN: now also U1.6 (UD-), U5.4 (I/O2)
- net USB_DP: now also U1.5 (UD+), U5.6 (I/O1)
- net VIN: now also J4.1, J5.2 (Pin_2), C22.1, TP1.1, U4.2 (EN), U4.3 (IN); no longer D7.1 (K)
- net VIN_RAW: no longer J4.1, J5.2 (Pin_2)
- net V_SENSE: now also U3.6 (IO34)
- net nDTR: now also U1.13 (~{DTR})
- net nRTS: now also U1.14 (~{RTS})
- net at C5.1, R5.2: now also U9.3 (Vs)
- net at R6.1: now also U1.2 (TXD)
- net at R7.1: now also U1.3 (RXD)
- net VBUS_FUSED: no longer names the net of F1.2
- net VBUS_FUSED: now also J6.1 (Pin_1)
- net VBUS_POSTFILTER renamed VBUS
- net VBUS: now also Q4.3 (D); no longer F1.1
- net VBUS_USBC renamed VBUS_RAW
- net VBUS_RAW: now also U5.5 (VBUS)
- new net: C24.1, R21.1, R22.2, U4.1 (FB)
- new net: C23.1, U4.6 (BST)
- new net: F4.2, J6.5 (Pin_5)
- new net: C20.1, F2.1, U8.5 (VOUT)
- new net BUCK_5V: C24.2, C25.1, C26.1, D6.2 (A), L2.2, Q4.1 (G), R11.1, R21.2, TP3.1
- new net BUCK_SW: C23.2, L2.1, U4.5 (SW)
- no-connect marks 22 -> 16
Other:
- note added: "ESP-WROOM-32E SoM"
- note added: "WS2812 Power & Data Output"
- note removed: "Buck Enable"
- note removed: "C_l = 2 * (C_load - C_stray)"
- note removed: "C_stray = 3-5 pF"
- note removed: "ESP-WROOM-32UE SoM"
- note removed: "ICS43434 or INMP441 I2S Microphone"
- note removed: "In case CH340C is used leave C1, C2, Y1 unpopulated"
- note removed: "WS2812 Data Output"
- moved on the sheet: C18, C21, D7, F1, F2
